File: kicad/project.sch (KiCad schematic (older format))
At the start: 37 parts, among them J1 Conn_01x05, J2 Conn_01x01, Q1 SI2323CDS, SW1 SW_SPDT, SW2 SW_SPDT, SW3 SW_Push, U1 STM32L031F4Px

Commit message: Also fit the premade mould from China
Parts:
- J2: footprint Mounting_Holes:MountingHole_2.5mm_Pad -> Mounting_Holes:MountingHole_2.2mm_M2_ISO7380_Pad
Changed lines of the file:
@@
 F 0 "J2" H 1975 4925 50  0000 C CNN
 F 1 "Conn_01x01" H 1975 4725 50  0000 C CNN
-F 2 "Mounting_Holes:MountingHole_2.5mm_Pad" H 1975 4825 50  0001 C CNN
+F 2 "Mounting_Holes:MountingHole_2.2mm_M2_ISO7380_Pad" H 1975 4825 50  0001 C CNN
 F 3 "" H 1975 4825 50  0001 C CNN
 	1    1975 4825

Commit message: Tidy up
Parts:
- R1: footprint Resistors_SMD:R_0805_HandSoldering -> Resistors_SMD:R_0603_HandSoldering
Changed lines of the file:
@@
 F 0 "R1" V 5030 3775 50  0000 C CNN
 F 1 "10K" V 4950 3775 50  0000 C CNN
-F 2 "Resistors_SMD:R_0805_HandSoldering" V 4880 3775 50  0001 C CNN
+F 2 "Resistors_SMD:R_0603_HandSoldering" V 4880 3775 50  0001 C CNN
 F 3 "" H 4950 3775 50  0001 C CNN
 	1    4950 3775

Commit message: Solder mask between pins of the stm32
Parts:
- U1: footprint Housings_SSOP:TSSOP-20_4.4x6.5mm_Pitch0.65mm -> theapi:TSSOP-20_4.4x6.5mm_Pitch0.65mm
Changed lines of the file:
@@
 F 0 "U1" H 5325 3025 50  0000 L BNN
 F 1 "STM32L031F4Px" H 6325 4875 50  0000 R BNN
-F 2 "Housings_SSOP:TSSOP-20_4.4x6.5mm_Pitch0.65mm" H 6675 2975 50  0001 R TNN
+F 2 "theapi:TSSOP-20_4.4x6.5mm_Pitch0.65mm" H 6675 2975 50  0001 R TNN
 F 3 "" H 5675 3925 50  0001 C CNN
 	1    5675 3925
